Commit message: added new plugin for mecanum wheels, slightly changed lidar position

File: VEXU_GHOST/ghost_description/urdf_robomasters/mecanum_macros.xacro (robot description, xacro)
@@ -6,32 +6,33 @@
             <visual>
                 <geometry>
-                    <cylinder radius="${wheel_radius}" length="${wheel_width}"/>
+                    <cylinder radius="${wheel_radius}" length="${wheel_width}" rpy="" />
                 </geometry>
                 <material name="black">
-                    <color rgba="0 0 0 1.0"/>
+                    <color rgba="0 0 0 1.0" />
                 </material>
             </visual>
             <collision>
-                <origin xyz="0 0 0"/>
+                <origin xyz="0 0 0" rpy="0.0 0.0 0.0"/>
                 <geometry>
-                    <cylinder radius="${wheel_radius}" length="${wheel_width}"/>
+                    <cylinder radius="${wheel_radius}" length="${wheel_width}" />
                 </geometry>
             </collision>
-            <!--Inertia estimated for solid cylinder of radius 2.5" and height 1" with mass 1 lb-->
+            <!--Inertia
+            estimated for solid cylinder of radius 2.5" and height 1" with mass 1 lb-->
             <!-- Just going with Maxx's math here and assuming swerve wheel ~ mecanum inertial-->
             <inertial>
-                <origin xyz="0 0 0"/>
-                <mass value="0.4545"/>
+                <origin xyz="0 0 0" />
+                <mass value="0.4545" />
                 <inertia
                     ixx="0.000482" ixy="0.0" ixz="0.0"
                     iyy="0.000482" iyz="0.0"
-                    izz="0.000914"/>
+                    izz="0.000914" />
             </inertial>
         </link>
         <joint name="base_${name}_joint" type="continuous">
-            <parent link="base_link"/>
-            <child link="${name}"/>
-            <origin xyz="${x_pos} ${y_pos} 0" rpy="-${pi/2} 0 0"/>
-            <axis xyz="0 0 1"/>
+            <parent link="base_link" />
+            <child link="${name}" />
+            <origin xyz="${x_pos} ${y_pos} 0" rpy="-${pi/2} 0 0" />
+            <axis xyz="0 0 1" />
         </joint>
     </xacro:macro>

File: VEXU_GHOST/ghost_description/urdf_robomasters/sentry.xacro (robot description, xacro)
@@ -79,4 +79,5 @@
         <origin xyz="0 0 0.25654"/>
     </joint>
+    <!-- importing all mecanum wheels from the macro files -->
     <xacro:mecanum_macro name="front_left_wheel" wheel_radius="${mecanum_diameter/2}" wheel_width="${mecanum_width}" x_pos="${x_dist_to_wheel}" y_pos="${y_dist_to_wheel}"/>
     <xacro:mecanum_macro name="front_right_wheel" wheel_radius="${mecanum_diameter/2}" wheel_width="${mecanum_width}" x_pos="${x_dist_to_wheel}" y_pos="-${y_dist_to_wheel}"/>

File: VEXU_GHOST/ghost_sim/urdf_robomasters/sentry_base.xacro (robot description, xacro)
@@ -1,22 +1,23 @@
 <?xml version="1.0"?>
 <robot name="sentry" xmlns:xacro="http://ros.org/wiki/xacro">
-    <xacro:include filename="$(find ghost_sim)/urdf/macros/actuator_macros.xacro"/>
-    <xacro:include filename="$(find ghost_sim)/urdf/macros/sensor_macros.xacro"/>
-    <!-- Import Primary Robot URDF -->
-    <xacro:include filename="$(find ghost_description)/urdf_robomasters/sentry.xacro"/>
-    <!-- Add Sensors -->
-    <xacro:lidar_macro link_name="lidar_link" topic_name="scan"></xacro:lidar_macro>
-    <!-- <xacro:imu_macro parent_link="camera_view_link"></xacro:imu_macro> -->
-    <!-- Add Mecanum -->
-    <!-- https://github.com/qaz9517532846/gazebo_mecanum_plugins/tree/ros2-foxy -->
-    <gazebo>
-      <plugin name="gazebo_ros_joint_state_publisher" filename="libgazebo_ros_joint_state_publisher.so">
-          <update_rate>100</update_rate>
-          <joint_name>base_back_left_wheel_joint</joint_name>
-          <joint_name>base_front_left_wheel_joint</joint_name>
-          <joint_name>base_front_right_wheel_joint</joint_name>
-          <joint_name>base_back_right_wheel_joint</joint_name>
-      </plugin>
-      <plugin name="gazebo_ros_mecanum_diff_drive" filename="libgazebo_mecanum_drive.so">
+  <xacro:include filename="$(find ghost_sim)/urdf/macros/actuator_macros.xacro" />
+  <xacro:include filename="$(find ghost_sim)/urdf/macros/sensor_macros.xacro" />
+  <!-- Import Primary Robot URDF -->
+  <xacro:include filename="$(find ghost_description)/urdf_robomasters/sentry.xacro" />
+  <!-- Add Sensors -->
+  <xacro:lidar_macro link_name="lidar_link" topic_name="scan"></xacro:lidar_macro>
+  <!-- <xacro:imu_macro parent_link="camera_view_link"></xacro:imu_macro> -->
+  <!-- Add Mecanum -->
+  <!-- https://github.com/qaz9517532846/gazebo_mecanum_plugins/tree/ros2-foxy -->
+  <gazebo>
+    <plugin name="gazebo_ros_joint_state_publisher"
+      filename="libgazebo_ros_joint_state_publisher.so">
+      <update_rate>100</update_rate>
+      <joint_name>base_back_left_wheel_joint</joint_name>
+      <joint_name>base_front_left_wheel_joint</joint_name>
+      <joint_name>base_front_right_wheel_joint</joint_name>
+      <joint_name>base_back_right_wheel_joint</joint_name>
+    </plugin>
+    <!-- <plugin name="gazebo_ros_mecanum_diff_drive" filename="libgazebo_mecanum_drive.so">
         <commandTopic>cmd_vel</commandTopic>
         <odometryTopic>odom</odometryTopic>
@@ -36,6 +37,41 @@
         <wheelDiameter>${mecanum_diameter}</wheelDiameter>
         <publishOdom>true</publishOdom>
-        <!-- <isRollerModel>true</isRollerModel> -->
+        <isRollerModel>true</isRollerModel>
+      </plugin> -->
+      <plugin name="differential_drive_controller" filename="libgazebo_ros_diff_drive.so">
+        <!-- Plugin update rate in Hz -->
+        <updateRate>100</updateRate>
+        <!-- Name of left joint, defaults to `left_joint` -->
+        <leftJoint>base_back_left_wheel_joint</leftJoint>
+        <!-- Name of right joint, defaults to `right_joint` -->
+        <rightJoint>base_back_right_wheel_joint</rightJoint>
+        <!-- The distance from the center of one wheel to the other, in meters, defaults to 0.34 m -->
+        <wheelSeparation>${2 * y_dist_to_wheel}</wheelSeparation>
+        <!-- Diameter of the wheels, in meters, defaults to 0.15 m -->
+        <wheelDiameter>${mecanum_diameter}</wheelDiameter>
+        <!-- Wheel acceleration, in rad/s^2, defaults to 0.0 rad/s^2 -->
+        <wheelAcceleration>5</wheelAcceleration>
+        <!-- Maximum torque which the wheels can produce, in Nm, defaults to 5 Nm -->
+        <wheelTorque>1</wheelTorque>
+        <!-- Topic to receive geometry_msgs/Twist message commands, defaults to `cmd_vel` -->
+        <commandTopic>cmd_vel</commandTopic>
+        <!-- Topic to publish nav_msgs/Odometry messages, defaults to `odom` -->
+        <odometryTopic>odom</odometryTopic>
+        <!-- Odometry frame, defaults to `odom` -->
+        <odometryFrame>odom</odometryFrame>
+        <!-- Robot frame to calculate odometry from, defaults to `base_footprint` -->
+        <robotBaseFrame>base_footprint</robotBaseFrame>
+        <!-- Odometry source, 0 for ENCODER, 1 for WORLD, defaults to WORLD -->
+        <odometrySource>1</odometrySource>
+        <!-- Set to true to publish transforms for the wheel links, defaults to false -->
+        <publishWheelTF>true</publishWheelTF>
+        <!-- Set to true to publish transforms for the odometry, defaults to true -->
+        <publishOdom>true</publishOdom>
+        <!-- Set to true to publish sensor_msgs/JointState on /joint_states for the wheel joints,
+        defaults to false -->
+        <publishWheelJointState>true</publishWheelJointState>
+        <!-- Set to true to swap right and left wheels, defaults to true -->
+        <legacyMode>false</legacyMode>
       </plugin>
-    </gazebo>
+  </gazebo>
 </robot>

Commit message: in progress

File: VEXU_GHOST/ghost_description/urdf_robomasters/mecanum_macros.xacro (robot description, xacro)
@@ -6,5 +6,5 @@
             <visual>
                 <geometry>
-                    <cylinder radius="${wheel_radius}" length="${wheel_width}" rpy="" />
+                    <cylinder radius="${wheel_radius}" length="${wheel_width}"/>
                 </geometry>
                 <material name="black">
@@ -13,5 +13,5 @@
             </visual>
             <collision>
-                <origin xyz="0 0 0" rpy="0.0 0.0 0.0"/>
+                <origin xyz="0 0 0"/>
                 <geometry>
                     <cylinder radius="${wheel_radius}" length="${wheel_width}" />
@@ -33,5 +33,5 @@
             <parent link="base_link" />
             <child link="${name}" />
-            <origin xyz="${x_pos} ${y_pos} 0" rpy="-${pi/2} 0 0" />
+            <origin xyz="${x_pos} ${y_pos} 0" rpy="${pi/2} 0 0" />
             <axis xyz="0 0 1" />
         </joint>

File: VEXU_GHOST/ghost_description/urdf_robomasters/sentry.xacro (robot description, xacro)
@@ -1,4 +1,7 @@
 <?xml version="1.0"?>
 <robot name="sentry" xmlns:xacro="http://ros.org/wiki/xacro">
+    <gazebo reference="base_link">
+        <pose>0 0 0 0 0 3.14</pose>
+    </gazebo>
     <xacro:include filename="$(find ghost_description)/urdf_robomasters/mecanum_macros.xacro"/>
     <xacro:property name="mecanum_diameter" value="0.1525"/>
@@ -39,5 +42,5 @@
     <link name="base_footprint">
         <inertial>
-            <origin xyz="0 0 0" rpy="0 0 0"/>
+            <origin xyz="0 0 0"/>
             <mass value="0.00001"/>
             <inertia
@@ -87,12 +90,12 @@
     <link name="lidar_link">
         <inertial>
-            <origin xyz="0.0 0 0.0" rpy="0 0 0"/>
+            <origin xyz="0 0 0"/>
             <mass value="0.125"/>
             <inertia ixx="0.001"  ixy="0"  ixz="0" iyy="0.001" iyz="0" izz="0.001" />
         </inertial>
         <visual>
-            <origin xyz="0 0 0" rpy="0 0 0"/>
+            <origin xyz="0 0 0"/>
             <geometry>
-            <cylinder radius="${0.06985/2}" length="0.0254"/>
+                <cylinder radius="${0.06985/2}" length="0.0254"/>
             </geometry>
         </visual>
@@ -101,5 +104,5 @@
         <parent link="base_link"/>
         <child link="lidar_link"/>
-        <origin xyz="0.098 0 0.22" rpy="0 0 0"/>
+        <origin xyz="0.098 0 0.22"/>
     </joint>
 </robot>

File: VEXU_GHOST/ghost_sim/urdf_robomasters/sentry_base.xacro (robot description, xacro)
@@ -19,59 +19,23 @@
       <joint_name>base_back_right_wheel_joint</joint_name>
     </plugin>
-    <!-- <plugin name="gazebo_ros_mecanum_diff_drive" filename="libgazebo_mecanum_drive.so">
-        <commandTopic>cmd_vel</commandTopic>
-        <odometryTopic>odom</odometryTopic>
-        <odometryFrame>world</odometryFrame>
-        <robotBaseFrame>base_footprint</robotBaseFrame>
-        <LeftRear>base_back_left_wheel_joint</LeftRear>
-        <LeftFront>base_front_left_wheel_joint</LeftFront>
-        <RightFront>base_front_right_wheel_joint</RightFront>
-        <RightRear>base_back_right_wheel_joint</RightRear>
-        <odometryRate>20</odometryRate>
-        <publishWheelTF>true</publishWheelTF>
-        <publishWheelJointState>true</publishWheelJointState>
-        <WheelTorque>1</WheelTorque>
-        <WheelSeparationW>${2 * y_dist_to_wheel}</WheelSeparationW>
-        <WheelSeparationL>${2 * x_dist_to_wheel}</WheelSeparationL>
-        <wheelAccel>5</wheelAccel>
-        <wheelDiameter>${mecanum_diameter}</wheelDiameter>
-        <publishOdom>true</publishOdom>
-        <isRollerModel>true</isRollerModel>
-      </plugin> -->
-      <plugin name="differential_drive_controller" filename="libgazebo_ros_diff_drive.so">
-        <!-- Plugin update rate in Hz -->
-        <updateRate>100</updateRate>
-        <!-- Name of left joint, defaults to `left_joint` -->
-        <leftJoint>base_back_left_wheel_joint</leftJoint>
-        <!-- Name of right joint, defaults to `right_joint` -->
-        <rightJoint>base_back_right_wheel_joint</rightJoint>
-        <!-- The distance from the center of one wheel to the other, in meters, defaults to 0.34 m -->
-        <wheelSeparation>${2 * y_dist_to_wheel}</wheelSeparation>
-        <!-- Diameter of the wheels, in meters, defaults to 0.15 m -->
-        <wheelDiameter>${mecanum_diameter}</wheelDiameter>
-        <!-- Wheel acceleration, in rad/s^2, defaults to 0.0 rad/s^2 -->
-        <wheelAcceleration>5</wheelAcceleration>
-        <!-- Maximum torque which the wheels can produce, in Nm, defaults to 5 Nm -->
-        <wheelTorque>1</wheelTorque>
-        <!-- Topic to receive geometry_msgs/Twist message commands, defaults to `cmd_vel` -->
-        <commandTopic>cmd_vel</commandTopic>
-        <!-- Topic to publish nav_msgs/Odometry messages, defaults to `odom` -->
-        <odometryTopic>odom</odometryTopic>
-        <!-- Odometry frame, defaults to `odom` -->
-        <odometryFrame>odom</odometryFrame>
-        <!-- Robot frame to calculate odometry from, defaults to `base_footprint` -->
-        <robotBaseFrame>base_footprint</robotBaseFrame>
-        <!-- Odometry source, 0 for ENCODER, 1 for WORLD, defaults to WORLD -->
-        <odometrySource>1</odometrySource>
-        <!-- Set to true to publish transforms for the wheel links, defaults to false -->
-        <publishWheelTF>true</publishWheelTF>
-        <!-- Set to true to publish transforms for the odometry, defaults to true -->
-        <publishOdom>true</publishOdom>
-        <!-- Set to true to publish sensor_msgs/JointState on /joint_states for the wheel joints,
-        defaults to false -->
-        <publishWheelJointState>true</publishWheelJointState>
-        <!-- Set to true to swap right and left wheels, defaults to true -->
-        <legacyMode>false</legacyMode>
-      </plugin>
+    <plugin name="mecanum_plugin" filename="libmecanum_plugin.so">
+      <LeftBack>base_back_left_wheel_joint</LeftBack>
+      <LeftFront>base_front_left_wheel_joint</LeftFront>
+      <RightFront>base_front_right_wheel_joint</RightFront>
+      <RightBack>base_back_right_wheel_joint</RightBack>
+      <BaseLink>base_link</BaseLink>
+      <WheelRadius>${mecanum_diameter/2}</WheelRadius>
+      <LeftRightSeperation>${2*x_dist_to_wheel}</LeftRightSeperation>
+      <FrontBackSeperation>${2*y_dist_to_wheel}</FrontBackSeperation>
+      <x_stddev>0.05</x_stddev>
+      <y_stddev>0.05</y_stddev>
+      <r_stddev>0.03</r_stddev>
+    </plugin>
+    <plugin name="object_controller" filename="libgazebo_ros_planar_move.so">
+      <commandTopic>mecanum_vel</commandTopic>
+      <publish_odom_tf>false</publish_odom_tf>
+      <publish_odom>false</publish_odom>
+      <robotBaseFrame>base_footprint</robotBaseFrame>
+    </plugin>
   </gazebo>
 </robot>

Commit message: fixes bugs in Mecanum plugin

File: VEXU_GHOST/ghost_description/urdf_robomasters/mecanum_macros.xacro (robot description, xacro)
@@ -33,5 +33,5 @@
             <parent link="base_link" />
             <child link="${name}" />
-            <origin xyz="${x_pos} ${y_pos} 0" rpy="${pi/2} 0 0" />
+            <origin xyz="${x_pos} ${y_pos} 0" rpy="${-pi/2} 0 0" />
             <axis xyz="0 0 1" />
         </joint>

File: VEXU_GHOST/ghost_description/urdf_robomasters/sentry.xacro (robot description, xacro)
@@ -2,9 +2,9 @@
 <robot name="sentry" xmlns:xacro="http://ros.org/wiki/xacro">
     <gazebo reference="base_link">
-        <pose>0 0 0 0 0 3.14</pose>
+        <pose>0 0 0 0 0 0.0</pose>
     </gazebo>
     <xacro:include filename="$(find ghost_description)/urdf_robomasters/mecanum_macros.xacro"/>
     <xacro:property name="mecanum_diameter" value="0.1525"/>
-    <xacro:property name="mecanum_width" value="0.04"/>
+    <xacro:property name="mecanum_width" value="0.0125"/>
     <xacro:property name="y_dist_to_wheel" value="0.183"/>
     <xacro:property name="x_dist_to_wheel" value="0.170"/>

File: VEXU_GHOST/ghost_sim/urdf_robomasters/sentry_base.xacro (robot description, xacro)
@@ -11,5 +11,5 @@
   <!-- https://github.com/qaz9517532846/gazebo_mecanum_plugins/tree/ros2-foxy -->
   <gazebo>
-    <plugin name="gazebo_ros_joint_state_publisher"
+    <!-- <plugin name="gazebo_ros_joint_state_publisher"
       filename="libgazebo_ros_joint_state_publisher.so">
       <update_rate>100</update_rate>
@@ -18,6 +18,59 @@
       <joint_name>base_front_right_wheel_joint</joint_name>
       <joint_name>base_back_right_wheel_joint</joint_name>
+    </plugin> -->
+    <plugin name="gazebo_mecanum_drive" filename="libgazebo_mecanum_drive.so">
+      <commandTopic>cmd_vel</commandTopic>
+      <odometryTopic>odom</odometryTopic>
+      <odometryFrame>odom</odometryFrame>
+      <robotBaseFrame>base_link</robotBaseFrame>
+      <LeftRear>base_back_left_wheel_joint</LeftRear>
+      <LeftFront>base_front_left_wheel_joint</LeftFront>
+      <RightFront>base_front_right_wheel_joint</RightFront>
+      <RightRear>base_back_right_wheel_joint</RightRear>
+      <odometryRate>20</odometryRate>
+      <publishWheelTF>true</publishWheelTF>
+      <publishWheelJointState>true</publishWheelJointState>
+      <WheelTorque>20.0</WheelTorque>
+      <WheelSeparationW>0.5</WheelSeparationW>
+      <WheelSeparationL>0.5</WheelSeparationL>
+      <wheelAccel>10.0</wheelAccel>
+      <wheelDiameter>0.13</wheelDiameter>
+      <publishOdom>true</publishOdom>
+      <publishOdomTF>true</publishOdomTF>
+      <isRollerModel>false</isRollerModel>
     </plugin>
-    <plugin name="mecanum_plugin" filename="libmecanum_plugin.so">
+    <!-- <plugin name="gazebo_mecanum_pid_drive" filename="libgazebo_mecanum_pid_drive.so">
+      <commandTopic>cmd_vel</commandTopic>
+      <odometryTopic>odom</odometryTopic>
+      <odometryFrame>odom</odometryFrame>
+      <robotBaseFrame>base_footprint</robotBaseFrame>
+      <LeftRear>base_back_left_wheel_joint</LeftRear>
+      <LeftFront>base_front_left_wheel_joint</LeftFront>
+      <RightFront>base_front_right_wheel_joint</RightFront>
+      <RightRear>base_back_right_wheel_joint</RightRear>
+      <odometryRate>20</odometryRate>
+      <publishWheelTF>true</publishWheelTF>
+      <publishOdomTF>true</publishOdomTF>
+      <WheelTorque>30</WheelTorque>
+      <WheelSeparationW>0.5</WheelSeparationW>
+      <WheelSeparationL>0.6</WheelSeparationL>
+      <wheelAccel>10</wheelAccel>
+      <wheelDiameter>0.13</wheelDiameter>
+      <publishOdom>true</publishOdom>
+      <isRollerModel>false</isRollerModel>
+      <Wheel_LR_P>10.0</Wheel_LR_P>
+      <Wheel_LR_I>0.0</Wheel_LR_I>
+      <Wheel_LR_D>0.0</Wheel_LR_D>
+      <Wheel_LF_P>10.0</Wheel_LF_P>
+      <Wheel_LF_I>0.0</Wheel_LF_I>
+      <Wheel_LF_D>0.0</Wheel_LF_D>
+      <Wheel_RF_P>10.0</Wheel_RF_P>
+      <Wheel_RF_I>0.0</Wheel_RF_I>
+      <Wheel_RF_D>0.0</Wheel_RF_D>
+      <Wheel_RR_P>10.0</Wheel_RR_P>
+      <Wheel_RR_I>0.0</Wheel_RR_I>
+      <Wheel_RR_D>0.0</Wheel_RR_D>
+    </plugin> -->
+    <!-- <plugin name="mecanum_plugin" filename="libmecanum_plugin.so">
       <LeftBack>base_back_left_wheel_joint</LeftBack>
       <LeftFront>base_front_left_wheel_joint</LeftFront>
@@ -37,5 +90,5 @@
       <publish_odom>false</publish_odom>
       <robotBaseFrame>base_footprint</robotBaseFrame>
-    </plugin>
+    </plugin> -->
   </gazebo>
 </robot>
