Commit message: particle filter working

File: VEXU_GHOST/ghost_description/urdf_robomasters/mecanum_macros.xacro (robot description, xacro)
@@ -23,9 +23,9 @@
             <inertial>
                 <origin xyz="0 0 0" />
-                <mass value="0.4545" />
+                <mass value="0.4545"/>
                 <inertia
-                    ixx="0.000482" ixy="0.0" ixz="0.0"
-                    iyy="0.000482" iyz="0.0"
-                    izz="0.000914" />
+                    ixx="0.000975" ixy="0.0" ixz="0.0"
+                    iyy="0.000975" iyz="0.0"
+                    izz="0.001902"/>
             </inertial>
         </link>

File: VEXU_GHOST/ghost_description/urdf_robomasters/sentry.xacro (robot description, xacro)
@@ -1,7 +1,4 @@
 <?xml version="1.0"?>
 <robot name="sentry" xmlns:xacro="http://ros.org/wiki/xacro">
-    <gazebo reference="base_link">
-        <pose>0 0 0 0 0 0.0</pose>
-    </gazebo>
     <xacro:include filename="$(find ghost_description)/urdf_robomasters/mecanum_macros.xacro"/>
     <xacro:property name="mecanum_diameter" value="0.1525"/>
@@ -16,12 +13,12 @@
             <origin xyz="0 0 0.1"/>
             <geometry>
-                <box size="0.47244 0.47244 0.2"/>
+                <box size="0.5 0.5 0.2"/>
             </geometry>
             <material name="see-through-silver"/>
         </visual>
         <collision>
-            <origin xyz="0 0 0.15"/>
+            <origin xyz="0 0 0.1"/>
             <geometry>
-                <box size="0.47244 0.47244 0.1"/>
+                <box size="0.5 0.5 0.2"/>
             </geometry>
         </collision>
@@ -29,10 +26,10 @@
         <!-- https://en.wikipedia.org/wiki/List_of_moments_of_inertia#List_of_3D_inertia_tensors -->
         <inertial>
-            <origin xyz="0 0 0"/>
-            <mass value="10"/>
+            <origin xyz="0 0 0.1"/>
+            <mass value="20"/>
             <inertia
-                ixx="0.240843" ixy="0.0" ixz="0.0"
-                iyy="0.240843" iyz="0.0"
-                izz="0.371997"/>
+                ixx="0.8333" ixy="0.0" ixz="0.0"
+                iyy="0.8333" iyz="0.0"
+                izz="0.4833"/>
         </inertial>
         <gazebo>

File: VEXU_GHOST/ghost_sim/urdf_robomasters/sentry_base.xacro (robot description, xacro)
@@ -11,16 +11,8 @@
   <!-- https://github.com/qaz9517532846/gazebo_mecanum_plugins/tree/ros2-foxy -->
   <gazebo>
-    <!-- <plugin name="gazebo_ros_joint_state_publisher"
-      filename="libgazebo_ros_joint_state_publisher.so">
-      <update_rate>100</update_rate>
-      <joint_name>base_back_left_wheel_joint</joint_name>
-      <joint_name>base_front_left_wheel_joint</joint_name>
-      <joint_name>base_front_right_wheel_joint</joint_name>
-      <joint_name>base_back_right_wheel_joint</joint_name>
-    </plugin> -->
     <plugin name="gazebo_mecanum_drive" filename="libgazebo_mecanum_drive.so">
       <commandTopic>cmd_vel</commandTopic>
       <odometryTopic>odom</odometryTopic>
-      <odometryFrame>odom</odometryFrame>
+      <odometryFrame>world</odometryFrame>
       <robotBaseFrame>base_link</robotBaseFrame>
       <LeftRear>base_back_left_wheel_joint</LeftRear>
@@ -40,55 +32,4 @@
       <isRollerModel>false</isRollerModel>
     </plugin>
-    <!-- <plugin name="gazebo_mecanum_pid_drive" filename="libgazebo_mecanum_pid_drive.so">
-      <commandTopic>cmd_vel</commandTopic>
-      <odometryTopic>odom</odometryTopic>
-      <odometryFrame>odom</odometryFrame>
-      <robotBaseFrame>base_footprint</robotBaseFrame>
-      <LeftRear>base_back_left_wheel_joint</LeftRear>
-      <LeftFront>base_front_left_wheel_joint</LeftFront>
-      <RightFront>base_front_right_wheel_joint</RightFront>
-      <RightRear>base_back_right_wheel_joint</RightRear>
-      <odometryRate>20</odometryRate>
-      <publishWheelTF>true</publishWheelTF>
-      <publishOdomTF>true</publishOdomTF>
-      <WheelTorque>30</WheelTorque>
-      <WheelSeparationW>0.5</WheelSeparationW>
-      <WheelSeparationL>0.6</WheelSeparationL>
-      <wheelAccel>10</wheelAccel>
-      <wheelDiameter>0.13</wheelDiameter>
-      <publishOdom>true</publishOdom>
-      <isRollerModel>false</isRollerModel>
-      <Wheel_LR_P>10.0</Wheel_LR_P>
-      <Wheel_LR_I>0.0</Wheel_LR_I>
-      <Wheel_LR_D>0.0</Wheel_LR_D>
-      <Wheel_LF_P>10.0</Wheel_LF_P>
-      <Wheel_LF_I>0.0</Wheel_LF_I>
-      <Wheel_LF_D>0.0</Wheel_LF_D>
-      <Wheel_RF_P>10.0</Wheel_RF_P>
-      <Wheel_RF_I>0.0</Wheel_RF_I>
-      <Wheel_RF_D>0.0</Wheel_RF_D>
-      <Wheel_RR_P>10.0</Wheel_RR_P>
-      <Wheel_RR_I>0.0</Wheel_RR_I>
-      <Wheel_RR_D>0.0</Wheel_RR_D>
-    </plugin> -->
-    <!-- <plugin name="mecanum_plugin" filename="libmecanum_plugin.so">
-      <LeftBack>base_back_left_wheel_joint</LeftBack>
-      <LeftFront>base_front_left_wheel_joint</LeftFront>
-      <RightFront>base_front_right_wheel_joint</RightFront>
-      <RightBack>base_back_right_wheel_joint</RightBack>
-      <BaseLink>base_link</BaseLink>
-      <WheelRadius>${mecanum_diameter/2}</WheelRadius>
-      <LeftRightSeperation>${2*x_dist_to_wheel}</LeftRightSeperation>
-      <FrontBackSeperation>${2*y_dist_to_wheel}</FrontBackSeperation>
-      <x_stddev>0.05</x_stddev>
-      <y_stddev>0.05</y_stddev>
-      <r_stddev>0.03</r_stddev>
-    </plugin>
-    <plugin name="object_controller" filename="libgazebo_ros_planar_move.so">
-      <commandTopic>mecanum_vel</commandTopic>
-      <publish_odom_tf>false</publish_odom_tf>
-      <publish_odom>false</publish_odom>
-      <robotBaseFrame>base_footprint</robotBaseFrame>
-    </plugin> -->
   </gazebo>
 </robot>
