Commit message: merge in dev changes

File: VEXU_GHOST/ghost_description/urdf/ghost1.xacro (robot description, xacro)
@@ -60,5 +60,5 @@
         <parent link="base_link"/>
         <child link="front_bar"/>
-        <origin xyz="0.175 0 0" rpy="0 0 0"/>
+        <origin xyz="0.156 0 0" rpy="0 0 0"/>
         <axis xyz="0 0 1"/>
     </joint>
@@ -77,5 +77,5 @@
         <parent link="base_link"/>
         <child link="left_bar"/>
-        <origin xyz="-0.05 0.125 0" rpy="0 0 -1.0471"/>
+        <origin xyz="-0.069 0.125 0" rpy="0 0 -1.0471"/>
         <axis xyz="0 0 1"/>
     </joint>
@@ -94,5 +94,5 @@
         <parent link="base_link"/>
         <child link="right_bar"/>
-        <origin xyz="-0.05 -0.125 0" rpy="0 0 1.0471"/>
+        <origin xyz="-0.069 -0.125 0" rpy="0 0 1.0471"/>
         <axis xyz="0 0 1"/>
     </joint>
@@ -109,5 +109,5 @@
         <parent link="base_link"/>
         <child link="mod_left"/>
-        <origin xyz="0.126365 0.180975 0.0812" rpy="0 0 0"/>
+        <origin xyz="0.10452 0.180975 0.0812" rpy="0 0 0"/>
         <axis xyz="0 0 1"/>
     </joint>
@@ -115,5 +115,5 @@
         <parent link="base_link"/>
         <child link="mod_right"/>
-        <origin xyz="0.126365 -0.180975 0.0812" rpy="0 0 0"/>
+        <origin xyz="0.10452 -0.180975 0.0812" rpy="0 0 0"/>
         <axis xyz="0 0 1"/>
     </joint>
@@ -121,5 +121,5 @@
         <parent link="base_link"/>
         <child link="mod_back"/>
-        <origin xyz="-0.187 0.0 0.0812" rpy="0 0 0"/>
+        <origin xyz="-0.209 0.0 0.0812" rpy="0 0 0"/>
         <axis xyz="0 0 1"/>
     </joint>
@@ -159,5 +159,5 @@
         <parent link="base_link"/>
         <child link="lidar_link"/>
-        <origin xyz="-0.19015 0 0.2145" rpy="0 0 0"/>
+        <origin xyz="-0.209 0 0.2145" rpy="0 0 ${67.562*d2r}"/>
     </joint>
     <!-- <link name="camera_base_link">
